File: Plane/PLANE.kicad_pcb (KiCad board)
At the start: 2 copper layers, 12 parts, among them Q1 2N3905, Q2 2N3906, SW1 SW_Push

Commit message: Add files via upload
Parts:
- moved BT1 87.7 mm to (165.1, 101.1)
- moved C1 87.7 mm to (126.1, 91.1)
- moved C2 87.7 mm to (126.1, 113.6)
- moved D1 87.7 mm to (123.6, 131.1)
- moved D2 87.7 mm to (123.6, 71.1)
- moved R2 87.7 mm to (131.1, 78.6)
- moved R3 87.7 mm to (143.6, 113.6)
- moved R4 87.7 mm to (143.5, 91.1)
- moved SW1 87.7 mm to (121.1, 98.6)
- moved Q1 87.7 mm to (126.1, 121.2)
- moved Q2 87.7 mm to (126.1, 83.7)
- moved R1 87.7 mm to (131.1, 123.5)
Other:
- board outline added: 100 x 107.5 mm
- board text added: "AEROPLANE"
- board text added: "BYE"
- board text added: "HELLO"
- board text removed: "my first pcb"

Commit message: Add files via upload
Parts:
- moved BT1 8.97 mm to (156.2, 100.0)
- moved D1 8.97 mm to (114.7, 130.0)
- moved D2 8.97 mm to (114.7, 70.0)
- moved R1 8.97 mm to (122.2, 122.4)
- moved C1 8.97 mm to (117.2, 90.0)
- moved C2 8.97 mm to (117.2, 112.5)
- moved Q1 8.97 mm to (117.2, 120.0)
- moved Q2 8.97 mm to (117.2, 82.5)
- moved R2 8.97 mm to (122.2, 77.5)
- moved SW1 8.97 mm to (112.2, 97.5)
- moved R3 8.97 mm to (134.7, 112.5)
- moved R4 8.97 mm to (134.6, 90.0)
Other:
- board size 100 x 107.5 mm -> 115 x 82.5 mm
- board text added: "KUSHINPI"
- board text added: "SUKHOI"
- board text removed: "AEROPLANE"
- board text removed: "BYE"
- board text removed: "HELLO"
